Commit message: Adjusted lidar position to remove interference with UAV frame. Smoothed UAV trajectory and tuned gains.

File: src/rbe594_asars/urdf/quadrotor_hokuyo_utm30lx_rotated.urdf.xacro (robot description, xacro)
@@ -8,6 +8,6 @@
     <!-- Hokuyo UTM-30LX mounted upside down below the quadrotor body -->
     <xacro:include filename="$(find hector_sensors_description)/urdf/hokuyo_utm30lx.urdf.xacro" />
-    <xacro:hokuyo_utm30lx name="laser0" parent="base_link" ros_topic="scan" update_rate="40" ray_count="100" min_angle="-60" max_angle="60">
-      <origin xyz="0 0.0 -0.097" rpy="${M_PI} ${M_PI/2} 0"/>
+    <xacro:hokuyo_utm30lx name="laser0" parent="base_link" ros_topic="scan" update_rate="30" ray_count="100" min_angle="-45" max_angle="45">
+      <origin xyz="0 0.0 -0.15" rpy="${M_PI} ${M_PI/2} 0"/>
     </xacro:hokuyo_utm30lx>
     <!-- Forward facing camera -->

Commit message: restructured GCS and victim spawning. Removed unneeded models from world

File: src/rbe594_asars/urdf/quadrotor_hokuyo_utm30lx_rotated.urdf.xacro (robot description, xacro)
@@ -9,5 +9,5 @@
     <xacro:include filename="$(find hector_sensors_description)/urdf/hokuyo_utm30lx.urdf.xacro" />
     <xacro:hokuyo_utm30lx name="laser0" parent="base_link" ros_topic="scan" update_rate="30" ray_count="100" min_angle="-45" max_angle="45">
-      <origin xyz="0 0.0 -0.15" rpy="${M_PI} ${M_PI/2} 0"/>
+      <origin xyz="0 0.0 -0.1" rpy="${M_PI} ${M_PI/2} 0"/>
     </xacro:hokuyo_utm30lx>
     <!-- Forward facing camera -->
